Commit message: added laser topic

File: description/lidar.xacro (robot description, xacro)
@@ -18,9 +18,9 @@
             </material>
         </visual>
-        <collision>
+        <!--<collision>
             <geometry>
                 <cylinder radius="0.05" length="0.04"/>
             </geometry>
-        </collision>
+        </collision>-->
         <xacro:inertial_cylinder mass="0.1" length="0.04" radius="0.05">
             <origin xyz="0 0 0" rpy="0 0 0"/>
@@ -33,4 +33,5 @@
             <visualize>true</visualize>
             <update_rate>10</update_rate>
+            <topic>scan</topic>
             <ray>
                 <scan>
